Commit message: finished

File: body.urdf (robot description, URDF)
Before this commit: robot robot, 9 links, 8 joints
Links:
- added link 10, mass 1.0; collision box size=0.6205379125824109 0.7529391823669973 0.6900473888648067; visual box size=0.6205379125824109 0.7529391823669973 0.6900473888648067
- added link 11, mass 1.0; collision box size=0.6205379125824109 0.7529391823669973 0.6900473888648067; visual box size=0.6205379125824109 0.7529391823669973 0.6900473888648067
- added link 12, mass 1.0; collision box size=0.6205379125824109 0.7529391823669973 0.6900473888648067; visual box size=0.6205379125824109 0.7529391823669973 0.6900473888648067
- added link 13, mass 1.0; collision box size=0.6205379125824109 0.7529391823669973 0.6900473888648067; visual box size=0.6205379125824109 0.7529391823669973 0.6900473888648067
- added link 14, mass 1.0; collision box size=0.6205379125824109 0.7529391823669973 0.6900473888648067; visual box size=0.6205379125824109 0.7529391823669973 0.6900473888648067
- added link 15, mass 1.0; collision box size=0.6205379125824109 0.7529391823669973 0.6900473888648067; visual box size=0.6205379125824109 0.7529391823669973 0.6900473888648067
- added link 16, mass 1.0; collision box size=0.6205379125824109 0.7529391823669973 0.6900473888648067; visual box size=0.6205379125824109 0.7529391823669973 0.6900473888648067
- added link 17, mass 1.0; collision box size=0.6205379125824109 0.7529391823669973 0.6900473888648067; visual box size=0.6205379125824109 0.7529391823669973 0.6900473888648067
- added link 18, mass 1.0; collision box size=0.6205379125824109 0.7529391823669973 0.6900473888648067; visual box size=0.6205379125824109 0.7529391823669973 0.6900473888648067
- added link 19, mass 1.0; collision box size=0.6205379125824109 0.7529391823669973 0.6900473888648067; visual box size=0.6205379125824109 0.7529391823669973 0.6900473888648067
- added link 9, mass 1.0; collision box size=0.6205379125824109 0.7529391823669973 0.6900473888648067; visual box size=0.6205379125824109 0.7529391823669973 0.6900473888648067
- link 0: geometry collision box size=0.5427232932533417 0.4981008313001189 0.5682431939992552; visual box size=0.5427232932533417 0.4981008313001189 0.5682431939992552
- link 1: geometry collision box size=0.5427232932533417 0.4981008313001189 0.5682431939992552; visual box size=0.5427232932533417 0.4981008313001189 0.5682431939992552
- link 2: geometry collision box size=0.5427232932533417 0.4981008313001189 0.5682431939992552; visual box size=0.5427232932533417 0.4981008313001189 0.5682431939992552
- link 3: geometry collision box size=0.5427232932533417 0.4981008313001189 0.5682431939992552; visual box size=0.5427232932533417 0.4981008313001189 0.5682431939992552
- link 4: geometry collision box size=0.5427232932533417 0.4981008313001189 0.5682431939992552; visual box size=0.5427232932533417 0.4981008313001189 0.5682431939992552
- link 5: geometry collision box size=0.6205379125824109 0.7529391823669973 0.6900473888648067; visual box size=0.6205379125824109 0.7529391823669973 0.6900473888648067
- link 6: geometry collision box size=0.6205379125824109 0.7529391823669973 0.6900473888648067; visual box size=0.6205379125824109 0.7529391823669973 0.6900473888648067
- link 7: geometry collision box size=0.6205379125824109 0.7529391823669973 0.6900473888648067; visual box size=0.6205379125824109 0.7529391823669973 0.6900473888648067
- link 8: geometry collision box size=0.6205379125824109 0.7529391823669973 0.6900473888648067; visual box size=0.6205379125824109 0.7529391823669973 0.6900473888648067
Joints:
- removed joint 7_8
- added joint 0_17: type revolute, parent 0, child 17, origin xyz=0.18403457564364956 -0.1295828239932062 2.4377072532280466 rpy=0 0 0, axis 0 0 1, limit lower=-3.14159 upper=3.14159 effort=0.0 velocity=0.0
- added joint 11_12: type revolute, parent 11, child 12, origin xyz=-0.01926427514057573 -0.5575295058168593 0.30471829264326605 rpy=0 0 0, axis 0 0 1, limit lower=-3.14159 upper=3.14159 effort=0.0 velocity=0.0
- added joint 12_13: type revolute, parent 12, child 13, origin xyz=0.14547928680402555 -0.4169471113688586 0.45762400058919467 rpy=0 0 0, axis 0 0 1, limit lower=-3.14159 upper=3.14159 effort=0.0 velocity=0.0
- added joint 14_15: type revolute, parent 14, child 15, origin xyz=0.312709673785332 -0.5502197829015657 -0.034438581497460534 rpy=0 0 0, axis 0 0 1, limit lower=-3.14159 upper=3.14159 effort=0.0 velocity=0.0
- added joint 15_16: type revolute, parent 15, child 16, origin xyz=0.4150643330960989 -0.4511838168276221 0.14931623234022057 rpy=0 0 0, axis 0 0 1, limit lower=-3.14159 upper=3.14159 effort=0.0 velocity=0.0
- added joint 17_18: type revolute, parent 17, child 18, origin xyz=0.5218905902803808 -0.33559947718370864 -0.08646968220998044 rpy=0 0 0, axis 0 0 1, limit lower=-3.14159 upper=3.14159 effort=0.0 velocity=0.0
- added joint 18_19: type revolute, parent 18, child 19, origin xyz=0.5569721023189039 -0.2783034453665202 0.0493388143524222 rpy=0 0 0, axis 0 0 1, limit lower=-3.14159 upper=3.14159 effort=0.0 velocity=0.0
- added joint 1_14: type revolute, parent 1, child 14, origin xyz=0.25763125412704474 -0.3404412753115185 -0.19279453748644743 rpy=0 0 0, axis 0 0 1, limit lower=-3.14159 upper=3.14159 effort=0.0 velocity=0.0
- added joint 2_11: type revolute, parent 2, child 11, origin xyz=-0.005751957539370495 -0.4771825271163619 0.0036453174887542544 rpy=0 0 0, axis 0 0 1, limit lower=-3.14159 upper=3.14159 effort=0.0 velocity=0.0
- added joint 3_8: type revolute, parent 3, child 8, origin xyz=-0.2535718962643009 -0.30919555350194206 0.2530201061107266 rpy=0 0 0, axis 0 0 1, limit lower=-3.14159 upper=3.14159 effort=0.0 velocity=0.0
- added joint 8_9: type revolute, parent 8, child 9, origin xyz=-0.3085894167097095 -0.17559836943066745 0.5213198226318037 rpy=0 0 0, axis 0 0 1, limit lower=-3.14159 upper=3.14159 effort=0.0 velocity=0.0
- added joint 9_10: type revolute, parent 9, child 10, origin xyz=-0.1625125288234221 -0.015971530015438447 0.6124544871364147 rpy=0 0 0, axis 0 0 1, limit lower=-3.14159 upper=3.14159 effort=0.0 velocity=0.0
- joint 0_1: origin xyz=-2.8606919601599716 0 2.5 rpy=0 0 0 -> xyz=0.27136164662667084 -0.23026603670960755 2.276264431415631 rpy=0 0 0
- joint 1_2: origin xyz=1.0483296597287202 0 0 rpy=0 0 0 -> xyz=0.21983211039922185 -0.4989462472249149 -0.23958753144456169 rpy=0 0 0
- joint 2_3: origin xyz=0.4143900996585757 0 0 rpy=0 0 0 -> xyz=-0.15412307296302957 -0.6059047221464934 0.07222860771766039 rpy=0 0 0
- joint 3_4: origin xyz=1.177863408926867 0 0 rpy=0 0 0 -> xyz=-0.42176881740977656 -0.2873151694016384 0.3414024054344654 rpy=0 0 0
- joint 4_5: origin xyz=0.6926911591473903 0 0 rpy=0 0 0 -> xyz=-0.3725077342015399 0.016545400948534697 0.27762140869497487 rpy=0 0 0
- joint 5_6: origin xyz=1.4907143750388925 0 0 rpy=0 0 0 -> xyz=-0.46923313529498634 0.2567732795424311 0.3253042818244062 rpy=0 0 0
- joint 6_7: origin xyz=0.9204342405929913 0 0 rpy=0 0 0 -> xyz=-0.37758195383826326 0.4094525663170668 0.29201235872696285 rpy=0 0 0

Commit message: readme

File: body.urdf (robot description, URDF)
Before this commit: robot robot, 20 links, 19 joints
Links:
- link 0: geometry collision box size=0.7042812383187429 0.48117543200991036 0.7213255229779734; visual box size=0.7042812383187429 0.48117543200991036 0.7213255229779734
- link 1: geometry collision box size=0.7042812383187429 0.48117543200991036 0.7213255229779734; visual box size=0.7042812383187429 0.48117543200991036 0.7213255229779734
- link 10: geometry collision box size=0.5772038644024104 0.900476230643817 0.4005201070583224; visual box size=0.5772038644024104 0.900476230643817 0.4005201070583224
- link 11: geometry collision box size=0.5772038644024104 0.900476230643817 0.4005201070583224; visual box size=0.5772038644024104 0.900476230643817 0.4005201070583224
- link 12: geometry collision box size=0.5772038644024104 0.900476230643817 0.4005201070583224; visual box size=0.5772038644024104 0.900476230643817 0.4005201070583224
- link 13: geometry collision box size=0.5772038644024104 0.900476230643817 0.4005201070583224; visual box size=0.5772038644024104 0.900476230643817 0.4005201070583224
- link 14: geometry collision box size=0.5772038644024104 0.900476230643817 0.4005201070583224; visual box size=0.5772038644024104 0.900476230643817 0.4005201070583224
- link 15: geometry collision box size=0.5772038644024104 0.900476230643817 0.4005201070583224; visual box size=0.5772038644024104 0.900476230643817 0.4005201070583224
- link 16: geometry collision box size=0.5772038644024104 0.900476230643817 0.4005201070583224; visual box size=0.5772038644024104 0.900476230643817 0.4005201070583224
- link 17: geometry collision box size=0.5772038644024104 0.900476230643817 0.4005201070583224; visual box size=0.5772038644024104 0.900476230643817 0.4005201070583224
- link 18: geometry collision box size=0.5772038644024104 0.900476230643817 0.4005201070583224; visual box size=0.5772038644024104 0.900476230643817 0.4005201070583224
- link 19: geometry collision box size=0.5772038644024104 0.900476230643817 0.4005201070583224; visual box size=0.5772038644024104 0.900476230643817 0.4005201070583224
- link 2: geometry collision box size=0.7042812383187429 0.48117543200991036 0.7213255229779734; visual box size=0.7042812383187429 0.48117543200991036 0.7213255229779734
- link 3: geometry collision box size=0.7042812383187429 0.48117543200991036 0.7213255229779734; visual box size=0.7042812383187429 0.48117543200991036 0.7213255229779734
- link 4: geometry collision box size=0.5772038644024104 0.900476230643817 0.4005201070583224; visual box size=0.5772038644024104 0.900476230643817 0.4005201070583224
- link 5: geometry collision box size=0.5772038644024104 0.900476230643817 0.4005201070583224; visual box size=0.5772038644024104 0.900476230643817 0.4005201070583224
- link 6: geometry collision box size=0.5772038644024104 0.900476230643817 0.4005201070583224; visual box size=0.5772038644024104 0.900476230643817 0.4005201070583224
- link 7: geometry collision box size=0.5772038644024104 0.900476230643817 0.4005201070583224; visual box size=0.5772038644024104 0.900476230643817 0.4005201070583224
- link 8: geometry collision box size=0.5772038644024104 0.900476230643817 0.4005201070583224; visual box size=0.5772038644024104 0.900476230643817 0.4005201070583224
- link 9: geometry collision box size=0.5772038644024104 0.900476230643817 0.4005201070583224; visual box size=0.5772038644024104 0.900476230643817 0.4005201070583224
Joints:
- removed joint 0_17
- removed joint 11_12
- removed joint 15_16
- removed joint 1_14
- removed joint 2_11
- removed joint 3_8
- added joint 0_16: type revolute, parent 0, child 16, origin xyz=0.19152949565024857 -0.22273729286812294 2.3298657273834804 rpy=0 0 0, axis 0 0 1, limit lower=-3.14159 upper=3.14159 effort=0.0 velocity=0.0
- added joint 10_11: type revolute, parent 10, child 11, origin xyz=0.10012315619231268 0.585723816496206 -0.101873742713107 rpy=0 0 0, axis 0 0 1, limit lower=-3.14159 upper=3.14159 effort=0.0 velocity=0.0
- added joint 13_14: type revolute, parent 13, child 14, origin xyz=0.0514429871915537 0.5763357835255618 -0.1736914202083345 rpy=0 0 0, axis 0 0 1, limit lower=-3.14159 upper=3.14159 effort=0.0 velocity=0.0
- added joint 16_17: type revolute, parent 16, child 17, origin xyz=0.2580609408337972 -0.49323911515945207 -0.21544995999198527 rpy=0 0 0, axis 0 0 1, limit lower=-3.14159 upper=3.14159 effort=0.0 velocity=0.0
- added joint 1_12: type revolute, parent 1, child 12, origin xyz=0.4318467176849012 0.28375507786761023 0.21824590038242123 rpy=0 0 0, axis 0 0 1, limit lower=-3.14159 upper=3.14159 effort=0.0 velocity=0.0
- added joint 2_8: type revolute, parent 2, child 8, origin xyz=0.497474120494715 0.09538533057992243 0.21696709506649497 rpy=0 0 0, axis 0 0 1, limit lower=-3.14159 upper=3.14159 effort=0.0 velocity=0.0
- joint 0_1: origin xyz=0.27136164662667084 -0.23026603670960755 2.276264431415631 rpy=0 0 0 -> xyz=0.35214061915937145 0.11314761475858054 2.6641007932382887 rpy=0 0 0
- joint 12_13: origin xyz=0.14547928680402555 -0.4169471113688586 0.45762400058919467 rpy=0 0 0 -> xyz=0.235358238140213 0.5439033981222967 0.07940439557281681 rpy=0 0 0
- joint 14_15: origin xyz=0.312709673785332 -0.5502197829015657 -0.034438581497460534 rpy=0 0 0 -> xyz=-0.13410362352988953 0.4258789210365372 -0.40941219478426244 rpy=0 0 0
- joint 17_18: origin xyz=0.5218905902803808 -0.33559947718370864 -0.08646968220998044 rpy=0 0 0 -> xyz=0.07778435186597589 -0.598322029530273 0.013050662852483382 rpy=0 0 0
- joint 18_19: origin xyz=0.5569721023189039 -0.2783034453665202 0.0493388143524222 rpy=0 0 0 -> xyz=-0.11015906230270728 -0.5258456193567878 0.28007315707174507 rpy=0 0 0
- joint 1_2: origin xyz=0.21983211039922185 -0.4989462472249149 -0.23958753144456169 rpy=0 0 0 -> xyz=0.6527239628132674 0.11111471622345094 0.2593417813829375 rpy=0 0 0
- joint 2_3: origin xyz=-0.15412307296302957 -0.6059047221464934 0.07222860771766039 rpy=0 0 0 -> xyz=0.68396749998949 -0.017079525904541107 0.1788673912318556 rpy=0 0 0
- joint 3_4: origin xyz=-0.42176881740977656 -0.2873151694016384 0.3414024054344654 rpy=0 0 0 -> xyz=0.525284121215979 -0.016612526410397146 0.1504152382368491 rpy=0 0 0
- joint 4_5: origin xyz=-0.3725077342015399 0.016545400948534697 0.27762140869497487 rpy=0 0 0 -> xyz=0.5031174474696998 0.10657975295244708 0.27372564868565813 rpy=0 0 0
- joint 5_6: origin xyz=-0.46923313529498634 0.2567732795424311 0.3253042818244062 rpy=0 0 0 -> xyz=0.43356723858421997 0.27397524854450567 0.28597642760058606 rpy=0 0 0
- joint 6_7: origin xyz=-0.37758195383826326 0.4094525663170668 0.29201235872696285 rpy=0 0 0 -> xyz=0.3166661609938959 0.46231386398223834 0.19705278863714262 rpy=0 0 0
- joint 8_9: origin xyz=-0.3085894167097095 -0.17559836943066745 0.5213198226318037 rpy=0 0 0 -> xyz=0.40760116606331065 0.334059671080107 0.26266497339922235 rpy=0 0 0
- joint 9_10: origin xyz=-0.1625125288234221 -0.015971530015438447 0.6124544871364147 rpy=0 0 0 -> xyz=0.2767306370089979 0.510391898990446 0.13476270851925595 rpy=0 0 0

Commit message: a better roll pitch yaw calculation

File: body.urdf (robot description, URDF)
Before this commit: robot robot, 20 links, 19 joints
Links:
- removed link 16
- removed link 17
- removed link 18
- removed link 19
- link 0: geometry collision box size=0.6840596376156676 0.7079142910708802 0.9407070144918339; visual box size=0.6840596376156676 0.7079142910708802 0.9407070144918339
- link 1: geometry collision box size=0.6840596376156676 0.7079142910708802 0.9407070144918339; visual box size=0.6840596376156676 0.7079142910708802 0.9407070144918339
- link 10: geometry collision box size=0.7835413528150419 0.5573811368381423 0.4818255872887541; visual box size=0.7835413528150419 0.5573811368381423 0.4818255872887541
- link 11: geometry collision box size=0.7835413528150419 0.5573811368381423 0.4818255872887541; visual box size=0.7835413528150419 0.5573811368381423 0.4818255872887541
- link 12: geometry collision box size=0.7835413528150419 0.5573811368381423 0.4818255872887541; visual box size=0.7835413528150419 0.5573811368381423 0.4818255872887541
- link 13: geometry collision box size=0.7835413528150419 0.5573811368381423 0.4818255872887541; visual box size=0.7835413528150419 0.5573811368381423 0.4818255872887541
- link 14: geometry collision box size=0.7835413528150419 0.5573811368381423 0.4818255872887541; visual box size=0.7835413528150419 0.5573811368381423 0.4818255872887541
- link 15: geometry collision box size=0.7835413528150419 0.5573811368381423 0.4818255872887541; visual box size=0.7835413528150419 0.5573811368381423 0.4818255872887541
- link 2: geometry collision box size=0.6840596376156676 0.7079142910708802 0.9407070144918339; visual box size=0.6840596376156676 0.7079142910708802 0.9407070144918339
- link 3: geometry collision box size=0.6840596376156676 0.7079142910708802 0.9407070144918339; visual box size=0.6840596376156676 0.7079142910708802 0.9407070144918339
- link 4: geometry collision box size=0.7835413528150419 0.5573811368381423 0.4818255872887541; visual box size=0.7835413528150419 0.5573811368381423 0.4818255872887541
- link 5: geometry collision box size=0.7835413528150419 0.5573811368381423 0.4818255872887541; visual box size=0.7835413528150419 0.5573811368381423 0.4818255872887541
- link 6: geometry collision box size=0.7835413528150419 0.5573811368381423 0.4818255872887541; visual box size=0.7835413528150419 0.5573811368381423 0.4818255872887541
- link 7: geometry collision box size=0.7835413528150419 0.5573811368381423 0.4818255872887541; visual box size=0.7835413528150419 0.5573811368381423 0.4818255872887541
- link 8: geometry collision box size=0.7835413528150419 0.5573811368381423 0.4818255872887541; visual box size=0.7835413528150419 0.5573811368381423 0.4818255872887541
- link 9: geometry collision box size=0.7835413528150419 0.5573811368381423 0.4818255872887541; visual box size=0.7835413528150419 0.5573811368381423 0.4818255872887541
Joints:
- removed joint 0_16
- removed joint 12_13
- removed joint 16_17
- removed joint 17_18
- removed joint 18_19
- removed joint 1_12
- removed joint 2_8
- removed joint 6_7
- removed joint 9_10
- added joint 0_13: type revolute, parent 0, child 13, origin xyz=0.09815735766491679 -0.18147275135556487 2.616903248208219 rpy=0 0 0, axis 0 0 1, limit lower=-3.14159 upper=3.14159 effort=0.0 velocity=0.0
- added joint 11_12: type revolute, parent 11, child 12, origin xyz=0.3865816646491185 -0.20762531444524515 -0.6570698054928462 rpy=0 0 0, axis 0 0 1, limit lower=-3.14159 upper=3.14159 effort=0.0 velocity=0.0
- added joint 1_10: type revolute, parent 1, child 10, origin xyz=0.3240554874734851 0.09412867765799768 -0.33515253107528875 rpy=0 0 0, axis 0 0 1, limit lower=-3.14159 upper=3.14159 effort=0.0 velocity=0.0
- added joint 2_7: type revolute, parent 2, child 7, origin xyz=0.04931999005817721 0.3808543565143046 -0.3030905961834568 rpy=0 0 0, axis 0 0 1, limit lower=-3.14159 upper=3.14159 effort=0.0 velocity=0.0
- added joint 7_8: type revolute, parent 7, child 8, origin xyz=0.2793102718354171 0.2870830117271478 -0.6824245089914274 rpy=0 0 0, axis 0 0 1, limit lower=-3.14159 upper=3.14159 effort=0.0 velocity=0.0
- joint 0_1: origin xyz=0.35214061915937145 0.11314761475858054 2.6641007932382887 rpy=0 0 0 -> xyz=0.3420298188078338 0.34273412340578147 2.1121621579335277 rpy=0 0 0
- joint 10_11: origin xyz=0.10012315619231268 0.585723816496206 -0.101873742713107 rpy=0 0 0 -> xyz=0.4806786509692844 -0.32134808814354243 -0.5366660349601625 rpy=0 0 0
- joint 13_14: origin xyz=0.0514429871915537 0.5763357835255618 -0.1736914202083345 rpy=0 0 0 -> xyz=0.2700879089117248 -0.6711090284015964 0.3208373819241639 rpy=0 0 0
- joint 14_15: origin xyz=-0.13410362352988953 0.4258789210365372 -0.40941219478426244 rpy=0 0 0 -> xyz=0.14680381618346405 -0.7625523713284654 0.15728545922678855 rpy=0 0 0
- joint 1_2: origin xyz=0.6527239628132674 0.11111471622345094 0.2593417813829375 rpy=0 0 0 -> xyz=0.10718776979190486 0.710309803877402 -0.3719775022709223 rpy=0 0 0
- joint 2_3: origin xyz=0.68396749998949 -0.017079525904541107 0.1788673912318556 rpy=0 0 0 -> xyz=-0.48043344926331516 0.691591587892214 0.14443115778483945 rpy=0 0 0
- joint 3_4: origin xyz=0.525284121215979 -0.016612526410397146 0.1504152382368491 rpy=0 0 0 -> xyz=-0.24748042853640456 0.38333349662264216 0.09721184253098573 rpy=0 0 0
- joint 4_5: origin xyz=0.5031174474696998 0.10657975295244708 0.27372564868565813 rpy=0 0 0 -> xyz=-0.10230557741204549 0.7840738466797083 -0.059584475539899956 rpy=0 0 0
- joint 5_6: origin xyz=0.43356723858421997 0.27397524854450567 0.28597642760058606 rpy=0 0 0 -> xyz=-0.22277787571263655 0.7476837127424416 0.13978460894253497 rpy=0 0 0
- joint 8_9: origin xyz=0.40760116606331065 0.334059671080107 0.26266497339922235 rpy=0 0 0 -> xyz=0.15677990579920004 0.46398716671267903 -0.6227470248109532 rpy=0 0 0
