Commit message: roll pitch yaw correction

File: body.urdf (robot description, URDF)
Before this commit: robot robot, 16 links, 15 joints
Links:
- added link 16, mass 1.0; collision box size=0.8583351681717986 0.24226134304531677 0.6073677863107836; visual box size=0.8583351681717986 0.24226134304531677 0.6073677863107836
- added link 17, mass 1.0; collision box size=0.8583351681717986 0.24226134304531677 0.6073677863107836; visual box size=0.8583351681717986 0.24226134304531677 0.6073677863107836
- link 0: geometry collision box size=0.46894964234140124 0.5097757701378711 0.9560491920449294; visual box size=0.46894964234140124 0.5097757701378711 0.9560491920449294
- link 1: geometry collision box size=0.46894964234140124 0.5097757701378711 0.9560491920449294; visual box size=0.46894964234140124 0.5097757701378711 0.9560491920449294
- link 10: geometry collision box size=0.8583351681717986 0.24226134304531677 0.6073677863107836; visual box size=0.8583351681717986 0.24226134304531677 0.6073677863107836
- link 11: geometry collision box size=0.8583351681717986 0.24226134304531677 0.6073677863107836; visual box size=0.8583351681717986 0.24226134304531677 0.6073677863107836
- link 12: geometry collision box size=0.8583351681717986 0.24226134304531677 0.6073677863107836; visual box size=0.8583351681717986 0.24226134304531677 0.6073677863107836
- link 13: geometry collision box size=0.8583351681717986 0.24226134304531677 0.6073677863107836; visual box size=0.8583351681717986 0.24226134304531677 0.6073677863107836
- link 14: geometry collision box size=0.8583351681717986 0.24226134304531677 0.6073677863107836; visual box size=0.8583351681717986 0.24226134304531677 0.6073677863107836
- link 15: geometry collision box size=0.8583351681717986 0.24226134304531677 0.6073677863107836; visual box size=0.8583351681717986 0.24226134304531677 0.6073677863107836
- link 2: geometry collision box size=0.46894964234140124 0.5097757701378711 0.9560491920449294; visual box size=0.46894964234140124 0.5097757701378711 0.9560491920449294
- link 3: geometry collision box size=0.8583351681717986 0.24226134304531677 0.6073677863107836; visual box size=0.8583351681717986 0.24226134304531677 0.6073677863107836
- link 4: geometry collision box size=0.8583351681717986 0.24226134304531677 0.6073677863107836; visual box size=0.8583351681717986 0.24226134304531677 0.6073677863107836
- link 5: geometry collision box size=0.8583351681717986 0.24226134304531677 0.6073677863107836; visual box size=0.8583351681717986 0.24226134304531677 0.6073677863107836
- link 6: geometry collision box size=0.8583351681717986 0.24226134304531677 0.6073677863107836; visual box size=0.8583351681717986 0.24226134304531677 0.6073677863107836
- link 7: geometry collision box size=0.8583351681717986 0.24226134304531677 0.6073677863107836; visual box size=0.8583351681717986 0.24226134304531677 0.6073677863107836
- link 8: geometry collision box size=0.8583351681717986 0.24226134304531677 0.6073677863107836; visual box size=0.8583351681717986 0.24226134304531677 0.6073677863107836
- link 9: geometry collision box size=0.8583351681717986 0.24226134304531677 0.6073677863107836; visual box size=0.8583351681717986 0.24226134304531677 0.6073677863107836
Joints:
- removed joint 1_10
- removed joint 2_7
- removed joint 7_8
- added joint 15_16: type revolute, parent 15, child 16, origin xyz=-0.8516809770968194 -0.01869457814269923 -0.1170929235353374 rpy=0 0 0, axis 0 0 1, limit lower=-3.14159 upper=3.14159 effort=0.0 velocity=0.0
- added joint 16_17: type revolute, parent 16, child 17, origin xyz=-0.857087376292356 -0.025753077888170404 -0.04460824456816974 rpy=0 0 0, axis 0 0 1, limit lower=-3.14159 upper=3.14159 effort=0.0 velocity=0.0
- added joint 1_8: type revolute, parent 1, child 8, origin xyz=-0.11991882189824866 -0.13177399831180814 0.06976703255476852 rpy=0 0 0, axis 0 0 1, limit lower=-3.14159 upper=3.14159 effort=0.0 velocity=0.0
- added joint 6_7: type revolute, parent 6, child 7, origin xyz=-0.8582978442063155 0.0035963455680038453 0.008157146150785534 rpy=0 0 0, axis 0 0 1, limit lower=-3.14159 upper=3.14159 effort=0.0 velocity=0.0
- added joint 9_10: type revolute, parent 9, child 10, origin xyz=-0.8476817488425198 -0.11106343801249716 -0.10036621842491456 rpy=0 0 0, axis 0 0 1, limit lower=-3.14159 upper=3.14159 effort=0.0 velocity=0.0
- joint 0_1: origin xyz=0.3420298188078338 0.34273412340578147 2.1121621579335277 rpy=0 0 0 -> xyz=0.23447482117070062 -0.16898551736257744 2.9151729358590712 rpy=0 0 0
- joint 0_13: origin xyz=0.09815735766491679 -0.18147275135556487 2.616903248208219 rpy=0 0 0 -> xyz=-0.18878047802908102 0.10805825591345074 2.3202930281515037 rpy=0 0 0
- joint 10_11: origin xyz=0.4806786509692844 -0.32134808814354243 -0.5366660349601625 rpy=0 0 0 -> xyz=-0.8563194546721674 -0.060900792863968475 -0.023940797081857035 rpy=0 0 0
- joint 11_12: origin xyz=0.3865816646491185 -0.20762531444524515 -0.6570698054928462 rpy=0 0 0 -> xyz=-0.8579611929552629 -0.02821294774051402 -9.172658010513004e-05 rpy=0 0 0
- joint 13_14: origin xyz=0.2700879089117248 -0.6711090284015964 0.3208373819241639 rpy=0 0 0 -> xyz=-0.7165176536953131 0.21982595449763065 -0.462762623162023 rpy=0 0 0
- joint 14_15: origin xyz=0.14680381618346405 -0.7625523713284654 0.15728545922678855 rpy=0 0 0 -> xyz=-0.8248040598822698 0.04627151777742495 -0.2581762053774729 rpy=0 0 0
- joint 1_2: origin xyz=0.10718776979190486 0.710309803877402 -0.3719775022709223 rpy=0 0 0 -> xyz=0.5433393389270514 0.04631933006734111 0.28338753411471956 rpy=0 0 0
- joint 2_3: origin xyz=-0.48043344926331516 0.691591587892214 0.14443115778483945 rpy=0 0 0 -> xyz=0.022949404881734244 0.03680710043344614 0.07160742054311994 rpy=0 0 0
- joint 3_4: origin xyz=-0.24748042853640456 0.38333349662264216 0.09721184253098573 rpy=0 0 0 -> xyz=-0.8525045740063035 -0.07131505059388613 0.08512223063709111 rpy=0 0 0
- joint 4_5: origin xyz=-0.10230557741204549 0.7840738466797083 -0.059584475539899956 rpy=0 0 0 -> xyz=-0.8572438621549004 -0.015659115633167575 0.0455588127781177 rpy=0 0 0
- joint 5_6: origin xyz=-0.22277787571263655 0.7476837127424416 0.13978460894253497 rpy=0 0 0 -> xyz=-0.8581331355761083 0.000860128557656045 0.020720968826002436 rpy=0 0 0
- joint 8_9: origin xyz=0.15677990579920004 0.46398716671267903 -0.6227470248109532 rpy=0 0 0 -> xyz=-0.8064758475757041 -0.15955855780502728 -0.2809910187045257 rpy=0 0 0

Commit message: streamlining code

File: body.urdf (robot description, URDF)
Before this commit: robot robot, 18 links, 17 joints
Links:
- added link 18, mass 1.0; collision box size=0.7687572737880206 0.9334496287658063 0.7455165027236428; visual box size=0.7687572737880206 0.9334496287658063 0.7455165027236428
- added link 19, mass 1.0; collision box size=0.7687572737880206 0.9334496287658063 0.7455165027236428; visual box size=0.7687572737880206 0.9334496287658063 0.7455165027236428
- added link 20, mass 1.0; collision box size=0.7687572737880206 0.9334496287658063 0.7455165027236428; visual box size=0.7687572737880206 0.9334496287658063 0.7455165027236428
- added link 21, mass 1.0; collision box size=0.7687572737880206 0.9334496287658063 0.7455165027236428; visual box size=0.7687572737880206 0.9334496287658063 0.7455165027236428
- added link 22, mass 1.0; collision box size=0.7687572737880206 0.9334496287658063 0.7455165027236428; visual box size=0.7687572737880206 0.9334496287658063 0.7455165027236428
- added link 23, mass 1.0; collision box size=0.7687572737880206 0.9334496287658063 0.7455165027236428; visual box size=0.7687572737880206 0.9334496287658063 0.7455165027236428
- added link 24, mass 1.0; collision box size=0.7687572737880206 0.9334496287658063 0.7455165027236428; visual box size=0.7687572737880206 0.9334496287658063 0.7455165027236428
- added link 25, mass 1.0; collision box size=0.7687572737880206 0.9334496287658063 0.7455165027236428; visual box size=0.7687572737880206 0.9334496287658063 0.7455165027236428
- added link 26, mass 1.0; collision box size=0.7687572737880206 0.9334496287658063 0.7455165027236428; visual box size=0.7687572737880206 0.9334496287658063 0.7455165027236428
- added link 27, mass 1.0; collision box size=0.7687572737880206 0.9334496287658063 0.7455165027236428; visual box size=0.7687572737880206 0.9334496287658063 0.7455165027236428
- added link 28, mass 1.0; collision box size=0.7687572737880206 0.9334496287658063 0.7455165027236428; visual box size=0.7687572737880206 0.9334496287658063 0.7455165027236428
- added link 29, mass 1.0; collision box size=0.7687572737880206 0.9334496287658063 0.7455165027236428; visual box size=0.7687572737880206 0.9334496287658063 0.7455165027236428
- link 0: geometry collision box size=0.21705524419809585 0.5964680199136614 0.43108951186840666; visual box size=0.21705524419809585 0.5964680199136614 0.43108951186840666
- link 1: geometry collision box size=0.21705524419809585 0.5964680199136614 0.43108951186840666; visual box size=0.21705524419809585 0.5964680199136614 0.43108951186840666
- link 10: geometry collision box size=0.7687572737880206 0.9334496287658063 0.7455165027236428; visual box size=0.7687572737880206 0.9334496287658063 0.7455165027236428
- link 11: geometry collision box size=0.7687572737880206 0.9334496287658063 0.7455165027236428; visual box size=0.7687572737880206 0.9334496287658063 0.7455165027236428
- link 12: geometry collision box size=0.7687572737880206 0.9334496287658063 0.7455165027236428; visual box size=0.7687572737880206 0.9334496287658063 0.7455165027236428
- link 13: geometry collision box size=0.7687572737880206 0.9334496287658063 0.7455165027236428; visual box size=0.7687572737880206 0.9334496287658063 0.7455165027236428
- link 14: geometry collision box size=0.7687572737880206 0.9334496287658063 0.7455165027236428; visual box size=0.7687572737880206 0.9334496287658063 0.7455165027236428
- link 15: geometry collision box size=0.7687572737880206 0.9334496287658063 0.7455165027236428; visual box size=0.7687572737880206 0.9334496287658063 0.7455165027236428
- link 16: geometry collision box size=0.7687572737880206 0.9334496287658063 0.7455165027236428; visual box size=0.7687572737880206 0.9334496287658063 0.7455165027236428
- link 17: geometry collision box size=0.7687572737880206 0.9334496287658063 0.7455165027236428; visual box size=0.7687572737880206 0.9334496287658063 0.7455165027236428
- link 2: geometry collision box size=0.21705524419809585 0.5964680199136614 0.43108951186840666; visual box size=0.21705524419809585 0.5964680199136614 0.43108951186840666
- link 3: geometry collision box size=0.21705524419809585 0.5964680199136614 0.43108951186840666; visual box size=0.21705524419809585 0.5964680199136614 0.43108951186840666
- link 4: geometry collision box size=0.21705524419809585 0.5964680199136614 0.43108951186840666; visual box size=0.21705524419809585 0.5964680199136614 0.43108951186840666
- link 5: geometry collision box size=0.7687572737880206 0.9334496287658063 0.7455165027236428; visual box size=0.7687572737880206 0.9334496287658063 0.7455165027236428
- link 6: geometry collision box size=0.7687572737880206 0.9334496287658063 0.7455165027236428; visual box size=0.7687572737880206 0.9334496287658063 0.7455165027236428
- link 7: geometry collision box size=0.7687572737880206 0.9334496287658063 0.7455165027236428; visual box size=0.7687572737880206 0.9334496287658063 0.7455165027236428
- link 8: geometry collision box size=0.7687572737880206 0.9334496287658063 0.7455165027236428; visual box size=0.7687572737880206 0.9334496287658063 0.7455165027236428
- link 9: geometry collision box size=0.7687572737880206 0.9334496287658063 0.7455165027236428; visual box size=0.7687572737880206 0.9334496287658063 0.7455165027236428
Joints:
- removed joint 0_13
- removed joint 14_15
- removed joint 1_8
- removed joint 9_10
- added joint 0_25: type revolute, parent 0, child 25, origin xyz=-0.06595253054611269 -0.2982340099568307 2.3087762169187442 rpy=0 0 0, axis 0 0 1, limit lower=-3.14159 upper=3.14159 effort=0.0 velocity=0.0
- added joint 12_13: type revolute, parent 12, child 13, origin xyz=0.48729101628467775 -0.3197902628759189 -0.5722959915960303 rpy=0 0 0, axis 0 0 1, limit lower=-3.14159 upper=3.14159 effort=0.0 velocity=0.0
- added joint 17_18: type revolute, parent 17, child 18, origin xyz=0.5100876463192237 0.37221062965817575 -0.5156181565538533 rpy=0 0 0, axis 0 0 1, limit lower=-3.14159 upper=3.14159 effort=0.0 velocity=0.0
- added joint 18_19: type revolute, parent 18, child 19, origin xyz=0.6815709182014662 0.015014087730699004 -0.4054505054259102 rpy=0 0 0, axis 0 0 1, limit lower=-3.14159 upper=3.14159 effort=0.0 velocity=0.0
- added joint 1_20: type revolute, parent 1, child 20, origin xyz=-0.08085844585908139 0.06590344401238946 0.2496961045035942 rpy=0 0 0, axis 0 0 1, limit lower=-3.14159 upper=3.14159 effort=0.0 velocity=0.0
- added joint 20_21: type revolute, parent 20, child 21, origin xyz=-0.2599491405637826 0.5320830875643646 0.5490866238196112 rpy=0 0 0, axis 0 0 1, limit lower=-3.14159 upper=3.14159 effort=0.0 velocity=0.0
- added joint 21_22: type revolute, parent 21, child 22, origin xyz=0.15481316957445052 0.7307892802711916 0.3465691033625019 rpy=0 0 0, axis 0 0 1, limit lower=-3.14159 upper=3.14159 effort=0.0 velocity=0.0
- added joint 22_23: type revolute, parent 22, child 23, origin xyz=0.5079776253502108 0.6378064590536114 -0.00373982375178444 rpy=0 0 0, axis 0 0 1, limit lower=-3.14159 upper=3.14159 effort=0.0 velocity=0.0
- added joint 23_24: type revolute, parent 23, child 24, origin xyz=0.6807724097409633 0.3378598848297977 -0.227620093577169 rpy=0 0 0, axis 0 0 1, limit lower=-3.14159 upper=3.14159 effort=0.0 velocity=0.0
- added joint 25_26: type revolute, parent 25, child 26, origin xyz=0.08869205262712171 -0.7667481747148869 -0.28348435817893974 rpy=0 0 0, axis 0 0 1, limit lower=-3.14159 upper=3.14159 effort=0.0 velocity=0.0
- added joint 26_27: type revolute, parent 26, child 27, origin xyz=0.4649107896913597 -0.6713259573388737 0.051911540164482316 rpy=0 0 0, axis 0 0 1, limit lower=-3.14159 upper=3.14159 effort=0.0 velocity=0.0
- added joint 27_28: type revolute, parent 27, child 28, origin xyz=0.6639682710463987 -0.35286632462805256 0.26300936291581883 rpy=0 0 0, axis 0 0 1, limit lower=-3.14159 upper=3.14159 effort=0.0 velocity=0.0
- added joint 28_29: type revolute, parent 28, child 29, origin xyz=0.7346315878577433 -0.056982232002740794 0.25666021369316977 rpy=0 0 0, axis 0 0 1, limit lower=-3.14159 upper=3.14159 effort=0.0 velocity=0.0
- added joint 2_15: type revolute, parent 2, child 15, origin xyz=-0.020352475371259997 0.18375574747660023 0.06691530003116354 rpy=0 0 0, axis 0 0 1, limit lower=-3.14159 upper=3.14159 effort=0.0 velocity=0.0
- added joint 3_10: type revolute, parent 3, child 10, origin xyz=0.007100050603568761 0.10338928507837229 -0.1092233068209222 rpy=0 0 0, axis 0 0 1, limit lower=-3.14159 upper=3.14159 effort=0.0 velocity=0.0
- added joint 7_8: type revolute, parent 7, child 8, origin xyz=0.44613332374306836 -0.6795109678363912 0.10209945210380846 rpy=0 0 0, axis 0 0 1, limit lower=-3.14159 upper=3.14159 effort=0.0 velocity=0.0
- joint 0_1: origin xyz=0.23447482117070062 -0.16898551736257744 2.9151729358590712 rpy=0 0 0 -> xyz=0.10852762209904793 -0.08940712165774557 2.586929060360666 rpy=0 0 0
- joint 10_11: origin xyz=-0.8563194546721674 -0.060900792863968475 -0.023940797081857035 rpy=0 0 0 -> xyz=-0.28783315461299935 0.21074154694529848 -0.7226628823034942 rpy=0 0 0
- joint 11_12: origin xyz=-0.8579611929552629 -0.02821294774051402 -9.172658010513004e-05 rpy=0 0 0 -> xyz=0.12227520970144284 -0.05661476317185789 -0.8118601785149279 rpy=0 0 0
- joint 13_14: origin xyz=-0.7165176536953131 0.21982595449763065 -0.462762623162023 rpy=0 0 0 -> xyz=0.6728230596465463 -0.37431968158520995 -0.19772740560891228 rpy=0 0 0
- joint 15_16: origin xyz=-0.8516809770968194 -0.01869457814269923 -0.1170929235353374 rpy=0 0 0 -> xyz=-0.25696012053155903 0.7586068800683698 -0.10464647582428996 rpy=0 0 0
- joint 16_17: origin xyz=-0.857087376292356 -0.025753077888170404 -0.04460824456816974 rpy=0 0 0 -> xyz=0.15821816561800273 0.7108325851802122 -0.38456353566915397 rpy=0 0 0
- joint 1_2: origin xyz=0.5433393389270514 0.04631933006734111 0.28338753411471956 rpy=0 0 0 -> xyz=0.19195966368299155 -0.0395120288119684 0.13248240047429297 rpy=0 0 0
- joint 2_3: origin xyz=0.022949404881734244 0.03680710043344614 0.07160742054311994 rpy=0 0 0 -> xyz=0.20795356556308445 0.06618028616809207 0.06366704503345794 rpy=0 0 0
- joint 3_4: origin xyz=-0.8525045740063035 -0.07131505059388613 0.08512223063709111 rpy=0 0 0 -> xyz=0.21264724854632783 0.060332334129984413 -0.028952251095964592 rpy=0 0 0
- joint 4_5: origin xyz=-0.8572438621549004 -0.015659115633167575 0.0455588127781177 rpy=0 0 0 -> xyz=0.020772198707498406 -0.05543601076119063 -0.10559438690489673 rpy=0 0 0
- joint 5_6: origin xyz=-0.8581331355761083 0.000860128557656045 0.020720968826002436 rpy=0 0 0 -> xyz=-0.33669587416651064 -0.5929944001281873 -0.42376468300684356 rpy=0 0 0
- joint 6_7: origin xyz=-0.8582978442063155 0.0035963455680038453 0.008157146150785534 rpy=0 0 0 -> xyz=0.06170669199237552 -0.7883899971108839 -0.22287113805902872 rpy=0 0 0
- joint 8_9: origin xyz=-0.8064758475757041 -0.15955855780502728 -0.2809910187045257 rpy=0 0 0 -> xyz=0.6563265576704997 -0.3462023294195 0.29341692899432736 rpy=0 0 0
